File: MIU60_REVB.brd (EAGLE design)
At the start: 546.1 x 63.5 mm, 80 parts, among them P1 PAD-10G, P2 PAD-10G

Commit message: Added the final piece in mechanical.lbr for final ground that I for some reason didnt add
Connections:
- net GND: now also U$10.GP4, U$11.GP4, U$12.GP4, U$13.GP4, U$14.GP4, U$9.GP4
Changed lines of the file:
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@@
 <wire x1="271.4286" y1="7.9036" x2="271.78" y2="8.255" width="1.016" layer="1"/>
 <via x="271.78" y="8.255" extent="1-16" drill="0.7"/>
+<contactref element="U$9" pad="GP4"/>
+<contactref element="U$10" pad="GP4"/>
+<contactref element="U$11" pad="GP4"/>
+<contactref element="U$12" pad="GP4"/>
+<contactref element="U$13" pad="GP4"/>
+<contactref element="U$14" pad="GP4"/>
 <wire x1="190.5" y1="7.9036" x2="190.5" y2="8.2536" width="0" layer="19" extent="1-1"/>
 <wire x1="444.5" y1="8.2536" x2="444.5" y2="7.9036" width="0" layer="19" extent="1-1"/>
